File: EMFbadge for MAKE/SMDEMFbadgeforMAKE-sizedfor3inchbagLCSCassembly/SMDEMFbadgeforMAKE-sizedfor3inchbagLCSCassembly.kicad_pcb (KiCad board)
At the start: 2 copper layers, 65 x 82.5 mm, 20 parts, among them J1 AudioJack2_Ground_Switch, SW1 SW_DPDT_x2, U1 NJM2115D

Commit message: EMFbadgework
Parts:
- AAA_Battery1, AAA_Battery2: footprint Battery:BatteryHolder_Keystone_2466_1xAAA -> Battery:AAA battery SMD
- C3, C4: value 10uF -> 1uF
- I1, I2: value 100mH -> 10mH
- J1: footprint Connector_Audio:Jack_3.5mm_CUI_SJ2-3593D-SMT_Horizontal -> Connector_Audio:Jack_3.5mm_CUI_SJ-3523-SMT_Horizontal
- U1: value NJM2115D -> MCP6002-E/P
- moved AAA_Battery1 22.3 mm to (222.4, 114.9)
- moved AAA_Battery2 22.2 mm to (185.6, 115.3)
- moved R1 15.3 mm to (214.4, 129.7)
- moved C1 14.9 mm to (209.1, 97.5), turned to 180 degrees
- moved C2 11.5 mm to (201.6, 97.4), turned to 0 degrees
- moved C3 9.13 mm to (195.9, 91.5), turned to 125 degrees
- moved R2 8.01 mm to (193.8, 130.8)
- moved C4 6.71 mm to (206.7, 89.8), turned to 35 degrees
- moved D1 4.72 mm to (204.2, 111.2)
- moved I1 4.63 mm to (193.0, 149.9), turned to 150 degrees
- moved R5 4.25 mm to (199.7, 114.9)
- moved I2 3.14 mm to (216.6, 149.5)
- moved C6 3.07 mm to (212.9, 103.7)
- moved R3 2.96 mm to (210.0, 103.8)
- moved U1 2.66 mm to (204.5, 104.2)
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Routing:
- net Net-(AAA_Battery1--): track 100.3 -> 0.00 mm
- net Net-(C2-Pad1): track 16.2 -> 0.00 mm
- net Net-(AAA_Battery2--): track 3.60 -> 0.00 mm
Other:
- board size 65 x 82.5 mm -> 65 x 86.7 mm
