File: EMFbadge for MAKE/SMDEMFbadgeforMAKE-sizedfor3inchbagLCSCassembly/SMDEMFbadgeforMAKE-sizedfor3inchbagLCSCassembly.kicad_sch (KiCad schematic)
At the start: 19 parts, among them J1 AudioJack2_Ground_Switch, SW1 SW_DPDT_x2, U1 NJM2115D

Commit message: EMFbadgework
Parts:
- C11, C2: value 10uF -> 1uF
- Inductor1, Inductor2: value 100mH -> 10mH
- U1: value NJM2115D -> MCP6002-E/P
Changed lines of the file:
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@@
 			)
 		)
-		(property "Value" "NJM2115D"
+		(property "Value" "MCP6002-E/P"
 			(at 135.89 88.9 0)
 			(effects
@@
 			)
 		)
-		(property "Value" "100mH"
+		(property "Value" "10mH"
 			(at 105.41 86.36 90)
 			(effects
@@
 			)
 		)
-		(property "Value" "NJM2115D"
+		(property "Value" "MCP6002-E/P"
 			(at 135.89 66.04 0)
 			(effects
@@
 			)
 		)
-		(property "Value" "10uF"
+		(property "Value" "1uF"
 			(at 160.02 71.12 0)
 			(effects
@@
 			)
 		)
-		(property "Value" "100mH"
+		(property "Value" "10mH"
 			(at 106.68 63.5 90)
 			(effects
@@
 			)
 		)
-		(property "Value" "NJM2115D"
+		(property "Value" "MCP6002-E/P"
 			(at 195.58 80.01 0)
 			(effects
@@
 			)
 		)
-		(property "Value" "10uF"
+		(property "Value" "1uF"
 			(at 160.02 95.25 0)
 			(effects

Commit message: PCBA assembly board work
Parts:
- AAA_BATT1: renamed from AAA_Battery1; value Spring_side-> -> AAA_BATT1; footprint Battery:BatteryHolder_Keystone_2466_1xAAA -> Battery:AAA battery SMD LCSC; LCSC C5290189 -> (none); THLCSC (none) -> C5290189
- AAA_BATT2: renamed from AAA_Battery2; value <-Spring_side -> AAA_BATT2; footprint Battery:BatteryHolder_Keystone_2466_1xAAA -> Battery:AAA battery SMD LCSC; LCSC C5290189 -> (none); THLCSC (none) -> C5290189
- C4: LCSC C216306 -> (none); SMDLCSC (none) -> C134741; THLCSC (none) -> C216306
- C6: LCSC C2896122 -> (none); SMDLCSC (none) -> C107172; THLCSC (none) -> C2896122
- D1: footprint LED_SMD:LED_Kingbright_APA1606_1.6x0.6mm_Horizontal -> LED_SMD:LED_0805_2012Metric_Pad1.15x1.40mm_HandSolder
- J1: footprint Connector_Audio:Jack_3.5mm_CUI_SJ2-3593D-SMT_Horizontal -> Connector_Audio:Jack_3.5mm_LCSC
- R3: LCSC C172965 -> (none); SMDLCSC (none) -> C17900; THLCSC (none) -> C172965
- SW1: footprint Button_Switch_SMD:SW_DPDT_CK_JS202011JCQN -> Button_Switch_SMD:SW_DPDT_LCSC
- U1: LCSC C640393 -> (none)
Changed lines of the file:
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@@
 			)
 		)
-		(property "LCSC" "C172965"
+		(property "THLCSC" "C172965"
 			(at 133.35 74.93 0)
+			(effects
+				(font
+					(size 1.27 1.27)
+				)
+				(hide yes)
+			)
+		)
+		(property "SMDLCSC" "C17900"
+			(at 135.89 72.39 90)
 			(effects
 				(font
@@
 			)
 		)
-		(property "LCSC" "C2896122"
+		(property "THLCSC" "C2896122"
 			(at 133.35 82.55 0)
+			(effects
+				(font
+					(size 1.27 1.27)
+				)
+				(hide yes)
+			)
+		)
+		(property "SMDLCSC" "C107172"
+			(at 135.89 78.74 90)
 			(effects
 				(font
@@
 		(property "Sim.Pins" "1=1 2=2 3=3 4=4 5=5"
 			(at 135.89 88.9 0)
-			(effects
-				(font
-					(size 1.27 1.27)
-				)
-				(hide yes)
-			)
-		)
-		(property "LCSC" "C640393"
-			(at 139.7 91.44 0)
 			(effects
 				(font
@@
 			)
 		)
-		(property "LCSC" "C640393"
-			(at 139.7 63.5 0)
-			(effects
-				(font
-					(size 1.27 1.27)
-				)
-				(hide yes)
-			)
-		)
 		(pin "1"
 		)
@@
 			)
 		)
-		(property "Footprint" "Button_Switch_SMD:SW_DPDT_CK_JS202011JCQN"
+		(property "Footprint" "Button_Switch_SMD:SW_DPDT_LCSC"
 			(at 231.14 76.2 0)
 			(effects
@@
 			)
 		)
-		(property "Footprint" "Connector_Audio:Jack_3.5mm_CUI_SJ2-3593D-SMT_Horizontal"
+		(property "Footprint" "Connector_Audio:Jack_3.5mm_LCSC"
 			(at 177.8 74.93 0)
 			(effects
@@
 			)
 		)
-		(property "LCSC" "C216306"
+		(property "THLCSC" "C216306"
 			(at 149.86 92.71 0)
+			(effects
+				(font
+					(size 1.27 1.27)
+				)
+				(hide yes)
+			)
+		)
+		(property "SMDLCSC" "C134741"
+			(at 149.86 88.9 90)
 			(effects
 				(font
@@
 		(property "Sim.Pins" "1=1 2=2 3=3 4=4 5=5"
 			(at 195.58 77.47 0)
-			(effects
-				(font
-					(size 1.27 1.27)
-				)
-				(hide yes)
-			)
-		)
-		(property "LCSC" "C640393"
-			(at 195.58 76.2 0)
 			(effects
 				(font
@@
 			)
 		)
-		(property "Footprint" "LED_SMD:LED_Kingbright_APA1606_1.6x0.6mm_Horizontal"
+		(property "Footprint" "LED_SMD:LED_0805_2012Metric_Pad1.15x1.40mm_HandSolder"
 			(at 204.47 74.93 0)
 			(effects
@@
 		(on_board yes)
 		(dnp no)
-		(property "Reference" "AAA_Battery1"
+		(property "Reference" "AAA_BATT1"
 			(at 219.71 85.09 0)
 			(effects
@@
 			)
 		)
-		(property "Value" "Spring_side->"
+		(property "Value" "AAA_BATT1"
 			(at 218.5417 83.947 0)
 			(effects
@@
 			)
 		)
-		(property "Footprint" "Battery:BatteryHolder_Keystone_2466_1xAAA"
+		(property "Footprint" "Battery:AAA battery SMD LCSC"
 			(at 222.25 85.344 90)
 			(effects
@@
 			)
 		)
-		(property "LCSC" "C5290189"
+		(property "THLCSC" "C5290189"
 			(at 219.71 85.09 0)
 			(effects
@@
 			)
 		)
+		(property "SMDLCSC" ""
+			(at 222.25 83.82 0)
+			(effects
+				(font
+					(size 1.27 1.27)
+				)
+				(hide yes)
+			)
+		)
 		(pin "1"
 		)
@@
 			(project "EMFbadge smallerforKitsNewLayout"
 				(path "/3f2d6e69-638e-4e7e-9e72-9aa39908357a"
-					(reference "AAA_Battery1")
+					(reference "AAA_BATT1")
 					(unit 1)
 				)
@@
 			)
 		)
-		(property "Footprint" "Button_Switch_SMD:SW_DPDT_CK_JS202011JCQN"
+		(property "Footprint" "Button_Switch_SMD:SW_DPDT_LCSC"
 			(at 213.36 66.04 0)
 			(effects
@@
 		(on_board yes)
 		(dnp no)
-		(property "Reference" "AAA_Battery2"
+		(property "Reference" "AAA_BATT2"
 			(at 219.71 72.39 0)
 			(effects
@@
 			)
 		)
-		(property "Value" "<-Spring_side"
+		(property "Value" "AAA_BATT2"
 			(at 218.5417 71.247 0)
 			(effects
@@
 			)
 		)
-		(property "Footprint" "Battery:BatteryHolder_Keystone_2466_1xAAA"
+		(property "Footprint" "Battery:AAA battery SMD LCSC"
 			(at 222.25 72.644 90)
 			(effects
@@
 			)
 		)
-		(property "LCSC" "C5290189"
+		(property "THLCSC" "C5290189"
 			(at 219.71 72.39 0)
 			(effects
 				(font
 					(size 1.27 1.27)
+					(italic yes)
+				)
+				(hide yes)
+			)
+		)
+		(property "SMDLCSC" ""
+			(at 222.25 71.12 0)
+			(effects
+				(font
+					(size 1.27 1.27)
 				)
 				(hide yes)
@@
 			(project "EMFbadge smallerforKitsNewLayout"
 				(path "/3f2d6e69-638e-4e7e-9e72-9aa39908357a"
-					(reference "AAA_Battery2")
-					(unit 1)
-				)
+					(reference "AAA_BATT2")
+					(unit 1)
+				)
