File: EMFbadge for MAKE/EMFbadgeforMAKE-sizedfor3inchbagLCSCassembly/EMFbadgeforMAKE-sizedfor3inchbagLCSCassembly.kicad_sch (KiCad schematic)
At the start: 19 parts, among them J1 AudioJack2_Ground_Switch, SW1 SW_DPDT_x2, U1 NJM2115D

Commit message: EMFbadgework
Parts:
- C11, C2: value 10uF -> 1uF
- Inductor1, Inductor2: value 100mH -> 10mH
- U1: value NJM2115D -> MCP6002-E/P
Changed lines of the file:
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@@
 			)
 		)
-		(property "Value" "NJM2115D"
+		(property "Value" "MCP6002-E/P"
 			(at 135.89 88.9 0)
 			(effects
@@
 			)
 		)
-		(property "Value" "100mH"
+		(property "Value" "10mH"
 			(at 105.41 86.36 90)
 			(effects
@@
 			)
 		)
-		(property "Value" "NJM2115D"
+		(property "Value" "MCP6002-E/P"
 			(at 135.89 66.04 0)
 			(effects
@@
 			)
 		)
-		(property "Value" "10uF"
+		(property "Value" "1uF"
 			(at 160.02 71.12 0)
 			(effects
@@
 			)
 		)
-		(property "Value" "100mH"
+		(property "Value" "10mH"
 			(at 106.68 63.5 90)
 			(effects
@@
 			)
 		)
-		(property "Value" "NJM2115D"
+		(property "Value" "MCP6002-E/P"
 			(at 195.58 80.01 0)
 			(effects
@@
 			)
 		)
-		(property "Value" "10uF"
+		(property "Value" "1uF"
 			(at 160.02 95.25 0)
 			(effects

Commit message: PCBA assembly board work
Parts:
- AAA_Battery1: LCSC (none) -> C5290189
- C11, C2: LCSC (none) -> C531341
- C3, C4: footprint Capacitor_THT:CP_Radial_D4.0mm_P2.54mm -> Capacitor_THT:CP_Radial_D4.0mm_P2.00mm; LCSC (none) -> C160645
- C5, C6: footprint Capacitor_THT:C_Disc_D3.4mm_W2.1mm_P2.50mm -> Capacitor_THT:C_Disc_D4.3mm_W1.9mm_P5.00mm; LCSC (none) -> C2896122
- D1, Inductor1, Inductor2: LCSC (none) -> NONE
- J1: LCSC (none) -> C4992449
- R1, R2: footprint Resistor_THT:R_Axial_DIN0207_L6.3mm_D2.5mm_P7.62mm_Horizontal -> Resistor_THT:R_Axial_DIN0207_L6.3mm_D2.5mm_P10.16mm_Horizontal; LCSC (none) -> C176450
- R3, R4: footprint Resistor_THT:R_Axial_DIN0207_L6.3mm_D2.5mm_P7.62mm_Horizontal -> Resistor_THT:R_Axial_DIN0207_L6.3mm_D2.5mm_P10.16mm_Horizontal; LCSC (none) -> C172965
- SW1: LCSC (none) -> C273399
- U1: value MCP6002-E/P -> MCP6002; LCSC (none) -> C640393
