File: EMFbadge for MAKE/EMFbadgeforMAKE-sizedfor3inchbagLCSCassembly/EMFbadgeforMAKE-sizedfor3inchbagLCSCassembly.kicad_pcb (KiCad board)
At the start: 2 copper layers, 65 x 82.5 mm, 19 parts, among them J1 AudioJack2_Ground_Switch, SW1 SW_DPDT_x2, U1 NJM2115D

Commit message: EMFbadgework
Parts:
- C1, C2: footprint Capacitor_THT:CP_Radial_D5.0mm_P2.00mm -> Capacitor_THT:CP_Radial_D4.0mm_P2.00mm
Routing:
- net GND: track 152.6 -> 157.4 mm
- net +VDC: track 23.0 -> 23.8 mm

Commit message: PCBA assembly board work
Parts:
- removed the AAA_Battery1 at (139.9, 134.0)
- added AAA_Battery2: <-Spring_side, Battery:BatteryHolder_Keystone_2466_1xAAA, B.Cu at (139.9, 134.1)
- added REF**: Tooling hole 1.152mm, MountingHole:Tooling Hole LCSC, F.Cu at (192.9, 134.3)
- added REF**: Tooling hole 1.152mm, MountingHole:Tooling Hole LCSC, F.Cu at (131.3, 134.2)
- C3, C4: value 10uF -> 1uF
- C5, C6: value 68pF -> 10pF
- I1, I2: value 100mH -> 10mH
- U1: value NJM2115D -> MCP6002
Other:
- board text added: "EMF Explorer badge V3a GitHub.com/Drc3p0"
- board text added: "SporkLogic.com"
- board text removed: "EMF badge LCSC assembled p1 /// SporkLogic"

Commit message: EMF badge files from MAKE
Routing:
- net +VDC: track 23.8 -> 22.2 mm
- net Net-(AAA_Battery2--): track 48.1 -> 49.6 mm
Other:
- outline, holes or cut-outs redrawn
- board text added: "EMF Explorer Badge V3a GitHub.com/Drc3p0"
- board text removed: "EMF Explorer badge V3a GitHub.com/Drc3p0"
Changed lines of the file:
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@@
 	)
 	(gr_line
-		(start 132.01 90.865)
-		(end 130.56 91.84)
+		(start 131.935 89.99)
+		(end 130.485 90.965)
 		(stroke
 			(width 0.2)
@@
 	)
 	(gr_circle
-		(center 161.585 74.69)
-		(end 159.68 74.69)
+		(center 161.935 74.54)
+		(end 160.03 74.54)
 		(stroke
 			(width 0.004398)
@@
 		(layer "Edge.Cuts")
 	)
-	(gr_text "EMF Explorer badge V3a GitHub.com/Drc3p0 "
-		(at 130.355 111.58 270)
+	(gr_text "EMF Explorer Badge V3a GitHub.com/Drc3p0 "
+		(at 130.285 110.79 270)
 		(layer "B.SilkS")
 		(effects
@@
 	)
 	(gr_text "Explore the electromagnetic fields around you"
-		(at 193.57255 111.481845 90)
+		(at 193.535 110.965 90)
 		(layer "B.SilkS")
 		(effects
@@
 	)
 	(segment
-		(start 172.054452 93.356797)
-		(end 173.207876 94.510221)
-		(width 0.5)
-		(layer "F.Cu")
-		(net 1)
-	)
-	(segment
 		(start 173.86 96.64)
 		(end 176.71 96.64)
@@
 	)
 	(segment
-		(start 171.520997 142.27)
-		(end 144.860799 142.27)
+		(start 136.433167 86.65801)
+		(end 140.774223 86.65801)
 		(width 0.5)
 		(layer "F.Cu")
@@
 	)
 	(segment
-		(start 136.433167 136.276301)
-		(end 136.433167 86.65801)
+		(start 172.054452 85.736797)
+		(end 172.054452 82.395548)
 		(width 0.5)
 		(layer "F.Cu")
@@
 	)
 	(segment
-		(start 140.044483 137.453684)
-		(end 137.61055 137.453684)
+		(start 145.892233 81.54)
+		(end 149.490127 81.54)
 		(width 0.5)
 		(layer "F.Cu")
@@
 	)
 	(segment
-		(start 172.054452 85.736797)
-		(end 172.054452 82.395548)
+		(start 137.61055 137.453684)
+		(end 136.433167 136.276301)
 		(width 0.5)
 		(layer "F.Cu")
@@
 	)
 	(segment
-		(start 136.433167 86.65801)
-		(end 140.774223 86.65801)
+		(start 140.774223 86.65801)
+		(end 145.892233 81.54)
 		(width 0.5)
 		(layer "F.Cu")
@@
 	)
 	(segment
-		(start 144.860799 142.27)
-		(end 140.044483 137.453684)
+		(start 171.520997 142.27)
+		(end 144.860799 142.27)
 		(width 0.5)
 		(layer "F.Cu")
@@
 	)
 	(segment
-		(start 137.61055 137.453684)
-		(end 136.433167 136.276301)
+		(start 149.490127 81.54)
+		(end 150.740127 80.29)
 		(width 0.5)
 		(layer "F.Cu")
@@
 	)
 	(segment
-		(start 171.7557 85.489634)
-		(end 166.870402 85.489634)
+		(start 140.044483 137.453684)
+		(end 137.61055 137.453684)
 		(width 0.5)
 		(layer "F.Cu")
@@
 	)
 	(segment
-		(start 140.774223 86.65801)
-		(end 147.142233 80.29)
+		(start 136.433167 136.276301)
+		(end 136.433167 86.65801)
 		(width 0.5)
 		(layer "F.Cu")
@@
 	)
 	(segment
-		(start 172.054452 82.395548)
-		(end 173.031668 81.418332)
+		(start 171.7557 85.489634)
+		(end 166.870402 85.489634)
 		(width 0.5)
 		(layer "F.Cu")
@@
 	)
 	(segment
-		(start 147.142233 80.29)
-		(end 150.740127 80.29)
+		(start 144.860799 142.27)
+		(end 140.044483 137.453684)
+		(width 0.5)
+		(layer "F.Cu")
+		(net 5)
+	)
+	(segment
+		(start 172.054452 82.395548)
+		(end 173.031668 81.418332)
 		(width 0.5)
 		(layer "F.Cu")
@@
 	)
 	(segment
-		(start 142.565295 82.044634)
-		(end 139.885 84.724929)
+		(start 163.474531 71.854531)
+		(end 160.731097 71.854531)
 		(width 0.5)
 		(layer "B.Cu")
@@
 	)
 	(segment
-		(start 166.805971 76.148359)
-		(end 162.684823 72.027211)
+		(start 174.223871 79.290265)
+		(end 170.852231 79.290265)
 		(width 0.5)
 		(layer "B.Cu")
@@
 	)
 	(segment
-		(start 160.066362 72.027211)
-		(end 155.570797 76.522776)
+		(start 160.731097 71.854531)
+		(end 156.062852 76.522776)
 		(width 0.5)
 		(layer "B.Cu")
@@
 	)
 	(segment
-		(start 170.538266 79.60423)
-		(end 170.852231 79.290265)
+		(start 174.281668 79.232468)
+		(end 174.179207 79.334929)
 		(width 0.5)
 		(layer "B.Cu")
@@
 	)
 	(segment
-		(start 174.281668 79.232468)
-		(end 174.179207 79.334929)
+		(start 170.852231 79.290265)
+		(end 170.538266 79.60423)
 		(width 0.5)
 		(layer "B.Cu")
@@
 	)
 	(segment
-		(start 152.123769 76.522776)
-		(end 142.565295 82.044634)
+		(start 139.885 84.724929)
+		(end 139.885 89.315)
 		(width 0.5)
 		(layer "B.Cu")
@@
 	)
 	(segment
-		(start 168.122688 79.60423)
-		(end 170.538266 79.60423)
+		(start 141.008706 84.724929)
+		(end 139.885 84.724929)
 		(width 0.5)
 		(layer "B.Cu")
@@
 	)
 	(segment
-		(start 170.852231 79.290265)
-		(end 174.223871 79.290265)
+		(start 166.805971 78.287513)
+		(end 166.805971 75.185971)
 		(width 0.5)
 		(layer "B.Cu")
@@
 	)
 	(segment
-		(start 166.805971 78.287513)
-		(end 166.805971 76.148359)
+		(start 166.805971 75.185971)
+		(end 163.474531 71.854531)
 		(width 0.5)
 		(layer "B.Cu")
@@
 	)
 	(segment
-		(start 174.223871 79.290265)
-		(end 174.281668 79.232468)
+		(start 149.935 77.89)
+		(end 147.31 80.515)
 		(width 0.5)
 		(layer "B.Cu")
@@
 	)
 	(segment
-		(start 139.885 84.724929)
-		(end 139.885 89.315)
+		(start 147.31 80.515)
+		(end 145.218635 80.515)
 		(width 0.5)
 		(layer "B.Cu")
@@
 	)
 	(segment
-		(start 166.805971 78.287513)
-		(end 168.122688 79.60423)
+		(start 151.81 77.89)
+		(end 149.935 77.89)
 		(width 0.5)
 		(layer "B.Cu")
@@
 	)
 	(segment
-		(start 155.570797 76.522776)
-		(end 152.123769 76.522776)
+		(start 145.218635 80.515)
+		(end 141.008706 84.724929)
 		(width 0.5)
 		(layer "B.Cu")
@@
 	)
 	(segment
-		(start 162.684823 72.027211)
-		(end 160.066362 72.027211)
+		(start 174.281668 79.232468)
+		(end 174.223871 79.290265)
+		(width 0.5)
+		(layer "B.Cu")
+		(net 15)
+	)
+	(segment
+		(start 156.062852 76.522776)
+		(end 153.177224 76.522776)
+		(width 0.5)
+		(layer "B.Cu")
+		(net 15)
+	)
+	(segment
+		(start 153.177224 76.522776)
+		(end 151.81 77.89)
+		(width 0.5)
+		(layer "B.Cu")
+		(net 15)
+	)
+	(segment
+		(start 168.122688 79.60423)
+		(end 166.805971 78.287513)
+		(width 0.5)
+		(layer "B.Cu")
+		(net 15)
+	)
+	(segment
+		(start 170.538266 79.60423)
+		(end 168.122688 79.60423)
 		(width 0.5)
 		(layer "B.Cu")
