File: SAOdumpsterfire/SAOdumpsterfire/SAOdumpsterfireSAOorPIN.kicad_pcb (KiCad board)
At the start: 2 copper layers, 40.9 x 51.9 mm, 5 parts, among them J2 SAO_header

Commit message: EMF PUSH
Parts:
- removed R1: R, Resistor_SMD:R_2010_5025Metric_Pad1.40x2.65mm_HandSolder
- moved D2 7.94 mm to (182.5, 102.7), turned to 40 degrees
- moved D1 6.30 mm to (157.4, 103.3), turned to -35 degrees
- moved BT1 0.65 mm to (168.9, 115.3)
- moved J2 0.11 mm to (169.5, 114.7)
Connections:
- D1 pad 1: Net-(D1-Pad1) -> Net-(BT1--)
- D2 pad 1: Net-(D2-Pad1) -> Net-(BT1--)
- D2 pad 2: Net-(D1-Pad1) -> Net-(BT1-+)
Routing:
- net Net-(D2-Pad1): track 17.2 -> 0.00 mm
- net Net-(BT1-+): track 30.3 -> 45.5 mm
- net Net-(BT1--): track 40.6 -> 53.1 mm
- net Net-(D1-Pad1): track 8.84 -> 0.00 mm
