File: SAOdumpsterfire/SAOdumpsterfire/SAOdumpsterfireSAOorPIN.kicad_sch (KiCad schematic)
At the start: 5 parts, among them J2 SAO_header

Commit message: EMF PUSH
Parts:
- removed R1: R, Resistor_SMD:R_2010_5025Metric_Pad1.40x2.65mm_HandSolder, symbol Device:R
Connections:
- net at BT1.1 (+), D1.2, J2.1 (VCC): now also D2.2
- net at BT1.2 (-), J2.2 (GND): now also D1.1, D2.1
Other:
- moved on the sheet: BT1, D1, D2
Changed lines of the file:
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@@
 	(paper "A4")
 	(junction
-		(at 85.09 100.33)
+		(at 83.82 99.06)
+		(diameter 0)
+		(color 0 0 0 0)
+	)
+	(junction
+		(at 83.82 90.17)
 		(diameter 0)
 		(color 0 0 0 0)
@@
 		(color 0 0 0 0)
 	)
-	(wire
-		(pts
-			(xy 83.82 100.33) (xy 85.09 100.33)
-		)
-		(stroke
-			(width 0)
-			(type default)
-		)
-	)
-	(wire
-		(pts
-			(xy 105.41 99.06) (xy 101.6 99.06)
+	(junction
+		(at 101.6 90.17)
+		(diameter 0)
+		(color 0 0 0 0)
+	)
+	(wire
+		(pts
+			(xy 83.82 99.06) (xy 83.82 90.17)
+		)
+		(stroke
+			(width 0)
+			(type default)
+		)
+	)
+	(wire
+		(pts
+			(xy 101.6 90.17) (xy 101.6 99.06)
+		)
+		(stroke
+			(width 0)
+			(type default)
+		)
+	)
+	(wire
+		(pts
+			(xy 96.52 83.82) (xy 101.6 83.82)
+		)
+		(stroke
+			(width 0)
+			(type default)
+		)
+	)
+	(wire
+		(pts
+			(xy 101.6 83.82) (xy 101.6 90.17)
 		)
 		(stroke
@@
 	(wire
 		(pts
-			(xy 100.33 87.63) (xy 105.41 87.63)
-		)
-		(stroke
-			(width 0)
-			(type default)
-		)
-	)
-	(wire
-		(pts
-			(xy 88.9 100.33) (xy 85.09 100.33)
-		)
-		(stroke
-			(width 0)
-			(type default)
-		)
-	)
-	(wire
-		(pts
-			(xy 105.41 87.63) (xy 105.41 91.44)
-		)
-		(stroke
-			(width 0)
-			(type default)
-		)
-	)
-	(wire
-		(pts
-			(xy 96.52 99.06) (xy 96.52 100.33)
-		)
-		(stroke
-			(width 0)
-			(type default)
-		)
-	)
-	(wire
-		(pts
-			(xy 85.09 100.33) (xy 85.09 87.63)
+			(xy 88.9 99.06) (xy 83.82 99.06)
+		)
+		(stroke
+			(width 0)
+			(type default)
+		)
+	)
+	(wire
+		(pts
+			(xy 96.52 90.17) (xy 101.6 90.17)
+		)
+		(stroke
+			(width 0)
+			(type default)
+		)
+	)
+	(wire
+		(pts
+			(xy 83.82 83.82) (xy 83.82 90.17)
 		)
 		(stroke
@@
 	(wire
 		(pts
-			(xy 83.82 107.95) (xy 83.82 100.33)
+			(xy 83.82 90.17) (xy 88.9 90.17)
+		)
+		(stroke
+			(width 0)
+			(type default)
+		)
+	)
+	(wire
+		(pts
+			(xy 83.82 99.06) (xy 83.82 107.95)
+		)
+		(stroke
+			(width 0)
+			(type default)
+		)
+	)
+	(wire
+		(pts
+			(xy 83.82 83.82) (xy 88.9 83.82)
 		)
 		(stroke
@@
 	(symbol
 		(lib_id "Device:Battery_Cell")
-		(at 93.98 100.33 90)
+		(at 93.98 99.06 90)
 		(unit 1)
 		(exclude_from_sim no)
@@
 		(on_board yes)
 		(dnp no)
-		(fields_autoplaced yes)
 		(property "Reference" "BT1"
-			(at 92.1385 92.71 90)
+			(at 95.758 97.79 90)
 			(effects
 				(font
@@
 		)
 		(property "Value" "Battery_Cell"
-			(at 92.1385 95.25 90)
+			(at 92.71 95.758 90)
 			(effects
 				(font
@@
 		)
 		(property "Footprint" "Battery:BatteryHolder_Keystone_1060_1x2032"
-			(at 92.456 100.33 90)
+			(at 92.456 99.06 90)
 			(effects
 				(font
@@
 		)
 		(property "Datasheet" "~"
-			(at 92.456 100.33 90)
+			(at 92.456 99.06 90)
 			(effects
 				(font
@@
 		)
 		(property "Description" "Single-cell battery"
-			(at 93.98 100.33 0)
+			(at 93.98 99.06 0)
 			(effects
 				(font
@@
 	(symbol
 		(lib_id "PCM_SL_Devices:LED_3mm")
-		(at 88.9 87.63 0)
+		(at 92.71 83.82 0)
 		(unit 1)
 		(exclude_from_sim no)
@@
 		(on_board yes)
 		(dnp no)
-		(fields_autoplaced yes)
 		(property "Reference" "D1"
-			(at 88.9 81.28 0)
+			(at 96.774 82.55 0)
 			(effects
 				(font
@@
 		)
 		(property "Value" "LED_3mm"
-			(at 88.9 83.82 0)
+			(at 92.964 80.772 0)
 			(effects
 				(font
@@
 		)
 		(property "Footprint" "LED_SMD:3mm LED sideways mount"
-			(at 87.884 90.424 0)
+			(at 91.694 86.614 0)
 			(effects
 				(font
@@
 		)
 		(property "Datasheet" ""
-			(at 87.63 87.63 0)
+			(at 91.44 83.82 0)
 			(effects
 				(font
@@
 		)
 		(property "Description" "3mm diameter small LED"
-			(at 88.9 87.63 0)
+			(at 92.71 83.82 0)
 			(effects
 				(font
@@
 	(symbol
 		(lib_id "PCM_SL_Devices:LED_3mm")
-		(at 96.52 87.63 0)
+		(at 92.71 90.17 0)
 		(unit 1)
 		(exclude_from_sim no)
@@
 		(on_board yes)
 		(dnp no)
-		(fields_autoplaced yes)
 		(property "Reference" "D2"
-			(at 96.52 81.28 0)
+			(at 97.028 89.154 0)
 			(effects
 				(font
@@
 		)
 		(property "Value" "LED_3mm"
-			(at 96.52 83.82 0)
+			(at 92.71 87.376 0)
 			(effects
 				(font
@@
 		)
 		(property "Footprint" "LED_SMD:3mm LED sideways mount"
-			(at 95.504 90.424 0)
+			(at 91.694 92.964 0)
 			(effects
 				(font
@@
 		)
 		(property "Datasheet" ""
-			(at 95.25 87.63 0)
+			(at 91.44 90.17 0)
 			(effects
 				(font
@@
 		)
 		(property "Description" "3mm diameter small LED"
-			(at 96.52 87.63 0)
+			(at 92.71 90.17 0)
 			(effects
 				(font
@@
 		(on_board yes)
 		(dnp no)
-		(fields_autoplaced yes)
 		(property "Reference" "J2"
-			(at 92.6611 101.6 90)
+			(at 95.504 101.092 90)
 			(effects
 				(font
@@
 		)
 		(property "Value" "SAO_header"
-			(at 92.6611 104.14 90)
+			(at 92.71 103.124 90)
 			(effects
 				(font
@@
 					(unit 1)
 				)
-			)
-		)
-	)
-	(symbol
-		(lib_id "Device:R")
-		(at 105.41 95.25 0)
-		(unit 1)
-		(exclude_from_sim no)
-		(in_bom yes)
-		(on_board yes)
-		(dnp no)
-		(fields_autoplaced yes)
-		(property "Reference" "R1"
-			(at 107.95 93.9799 0)
-			(effects
-				(font
-					(size 1.27 1.27)
-				)
-				(justify left)
-			)
-		)
-		(property "Value" "R"
-			(at 107.95 96.5199 0)
-			(effects
-				(font
-					(size 1.27 1.27)
-				)
-				(justify left)
-			)
-		)
-		(property "Footprint" "Resistor_SMD:R_2010_5025Metric_Pad1.40x2.65mm_HandSolder"
-			(at 103.632 95.25 90)
-			(effects
-				(font
-					(size 1.27 1.27)
-				)
-				(hide yes)
-			)
-		)
-		(property "Datasheet" "~"
-			(at 105.41 95.25 0)
-			(effects
-				(font
-					(size 1.27 1.27)
-				)
-				(hide yes)
-			)
-		)
-		(property "Description" "Resistor"
-			(at 105.41 95.25 0)
-			(effects
-				(font
-					(size 1.27 1.27)
-				)
-				(hide yes)
-			)
-		)
-		(pin "1"
-		)
-		(pin "2"
-		)
-		(instances
-			(project ""
-				(path "/d26d2ec8-25fa-4775-aa69-f16b8aecde20"
-					(reference "R1")
-					(unit 1)
-				)
